File: Phase B - Copy - Copy/Uno_Shield_ThermoPro_Jeremy_trafas/Uno_Shield_ThermoPro.kicad_pcb (KiCad board)
At the start: 2 copper layers, 68.6 x 53.3 mm, 20 parts, among them J1 Power, J2 Digital/PWM, J3 Analog, J4 Digital/PWM, J5 CONN_GYRO, J6 CONN_DISPLAY, J7 CONN_TEMP, SW1 SW_SPST, SW2 SW_SPST, SW3 SW_SPST, SW4 SW_SPST, SW5 SW_SPST

Commit message: Update PCB
Routing:
- net /button_light: track 148.8 -> 152.4 mm
Other:
- board text added: "ANALOG SENSOR"
- board text added: "CAL"
- board text added: "Jeremy Trafas 2/3/25 V1"
- board text added: "LIGHT"
- board text added: "LOCK"
- board text added: "MPU6050"
- board text added: "OLED"
- board text added: "ON/OFF"
- board text added: "TEMP SENSOR"
- board text added: "UNITS"

Commit message: Update PCB
Routing:
- net +5V: track 130.4 -> 135.8 mm
- net /button_light: track 152.4 -> 149.6 mm
- net Net-(D1-A): track 43.7 -> 42.7 mm
- net /led_light: track 36.0 -> 35.4 mm
- net /I2C_SCL: track 28.6 -> 28.0 mm
- net /I2C_SDA: track 28.2 -> 27.7 mm

Commit message: Fixed PCB
Changed lines of the file:
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@@
 		(grid_origin 100 100)
 		(pcbplotparams
-			(layerselection 0x0000030_80000001)
+			(layerselection 0x00010fc_ffffffff)
 			(plot_on_all_layers_selection 0x0000000_00000000)
 			(disableapertmacros no)
@@
 			(outputformat 1)
 			(mirror no)
-			(drillshape 1)
+			(drillshape 0)
 			(scaleselection 1)
-			(outputdirectory "")
+			(outputdirectory "gerber/")
 		)
 	)
@@
 	)
 	(segment
-		(start 147.946067 94.470067)
-		(end 155.750207 86.665927)
+		(start 136.984256 51.331181)
+		(end 136.985153 51.330284)
 		(width 0.508)
 		(layer "F.Cu")
@@
 	)
 	(segment
-		(start 144.085786 84.414213)
-		(end 141 87.5)
+		(start 147.946067 94.470067)
+		(end 155.750207 86.665927)
 		(width 0.508)
 		(layer "F.Cu")
@@
 	)
 	(segment
-		(start 126.5 57.100589)
-		(end 126.5 61.786877)
+		(start 144.085786 84.414213)
+		(end 141 87.5)
 		(width 0.508)
 		(layer "F.Cu")
@@
 	)
 	(segment
-		(start 126.5 55.636543)
-		(end 126.5 57.100589)
-		(width 0.508)
-		(layer "F.Cu")
-		(net 25)
-	)
-	(segment
-		(start 126.5 69.5)
-		(end 126.5 61.786877)
-		(width 0.508)
-		(layer "F.Cu")
-		(net 25)
-	)
-	(segment
 		(start 146.914213 77.585786)
 		(end 148.116324 76.383675)
@@
 	)
 	(segment
+		(start 126.5 57.100589)
+		(end 126.5 55.636543)
+		(width 0.508)
+		(layer "F.Cu")
+		(net 25)
+	)
+	(segment
 		(start 141 87.5)
 		(end 134.5 87.5)
@@
 	)
 	(segment
-		(start 131.241702 50.894841)
-		(end 138.894841 50.894841)
+		(start 126.5 69.5)
+		(end 126.5 57.100589)
 		(width 0.508)
 		(layer "F.Cu")
@@
 	)
 	(segment
+		(start 131.678042 51.331181)
+		(end 136.984256 51.331181)
+		(width 0.508)
+		(layer "F.Cu")
+		(net 25)
+	)
+	(segment
+		(start 131.241702 50.894841)
+		(end 131.678042 51.331181)
+		(width 0.508)
+		(layer "F.Cu")
+		(net 25)
+	)
+	(segment
 		(start 143.584015 51.5)
 		(end 140.5 51.5)
@@
 	)
 	(via
-		(at 138.894841 50.894841)
+		(at 137 51.5)
 		(size 0.6)
 		(drill 0.4)
@@
 	)
 	(arc
-		(start 144.884261 52.038579)
-		(mid 144.287703 51.639972)
-		(end 143.584015 51.5)
+		(start 126.5 55.636543)
+		(mid 126.86094 53.821972)
+		(end 127.888812 52.283653)
 		(width 0.508)
 		(layer "F.Cu")
@@
 	)
 	(arc
-		(start 127.888812 52.283653)
-		(mid 126.86094 53.821972)
-		(end 126.5 55.636543)
+		(start 144.884261 52.038579)
+		(mid 144.287703 51.639972)
+		(end 143.584015 51.5)
 		(width 0.508)
 		(layer "F.Cu")
@@
 	)
 	(arc
+		(start 127.888812 52.283653)
+		(mid 129.427131 51.255781)
+		(end 131.241702 50.894841)
+		(width 0.508)
+		(layer "F.Cu")
+		(net 25)
+	)
+	(arc
 		(start 157.344 82.818171)
 		(mid 156.929786 84.900561)
@@
 	)
 	(arc
-		(start 131.241702 50.894841)
-		(mid 129.427131 51.255781)
-		(end 127.888812 52.283653)
-		(width 0.508)
-		(layer "F.Cu")
-		(net 25)
-	)
-	(arc
 		(start 146.690918 50.769081)
 		(mid 146.549617 50.980552)
@@
 	)
 	(segment
-		(start 126.5 71.068)
-		(end 126.5 69.5)
+		(start 138.00165 50.896491)
+		(end 137.603509 50.896491)
 		(width 0.508)
 		(layer "B.Cu")
@@
 	)
 	(segment
-		(start 139.466928 50.894841)
-		(end 138.894841 50.894841)
+		(start 140.5 51.5)
+		(end 140.19742 51.19742)
 		(width 0.508)
 		(layer "B.Cu")
@@
 	)
 	(segment
-		(start 140.19742 51.19742)
-		(end 140.5 51.5)
+		(start 137.603509 50.896491)
+		(end 137 51.5)
+		(width 0.508)
+		(layer "B.Cu")
+		(net 25)
+	)
+	(segment
+		(start 126.5 71.068)
+		(end 126.5 69.5)
+		(width 0.508)
+		(layer "B.Cu")
+		(net 25)
+	)
+	(segment
+		(start 139.568513 50.896491)
+		(end 138.00165 50.896491)
 		(width 0.508)
 		(layer "B.Cu")
@@
 	(arc
 		(start 140.19742 51.19742)
-		(mid 139.862267 50.973478)
-		(end 139.466928 50.894841)
+		(mid 139.908625 50.994016)
+		(end 139.568513 50.896491)
 		(width 0.508)
 		(layer "B.Cu")
